File: 1.UberDirver v2 + Sensory v2/Sam sterownik/Schematic.brd (EAGLE design)
At the start: 271.8 x 122.6 mm, 159 parts, among them IC1 MCP23017ML, IC2 TPS70933DBV, IC3 LM2596S, IC4 ACS758ECB-200B-PFF-T, U1 VL53L0X, U2 STM32F10XTXU6HS, U3 STM32F10XRXT6

Commit message: Wersja 3
Parts:
- removed 0003, 0010, 0012, 0013, 0030, 0031: 10k, resistor:R0603
- removed 0004: 26.1k, resistor:R0603
- removed 0005: 6.8k, resistor:R0603
- removed 0006, 0007, 0008, 0011, 0022, 0023, 0025, 0027, 0028: 100k, resistor:R0603
- removed 0009: 1k, resistor:R0603
- removed 0024: 300k, resistor:R0603
- removed 0026: 500k, resistor:R0603
- removed 0029: 700k, resistor:R0603
- removed 0032, 0033: ?, resistor:R0603
- removed C18, C21: 10nF, rcl:C0603
- removed C19, C20, C23: (no value), rcl:153CLV-0810
- removed C22, C27: 100nF, rcl:C0603
- removed C24: 3.9nF, rcl:C0603
- removed C25: 22uF, rcl:C0805
- removed C26: 10uF, rcl:153CLV-0605
- removed C28, C29: 10uF, rcl:C0805
- removed C30: 10uF/10V, rcl:SMC_A
- removed C33: 10uf/10V, rcl:SMC_A
- removed C35: (no value), rcl:C0603
- removed D1: (no value), diode:SMB
- removed DIODE: (no value), rcl:R0805
- removed IC1: MCP23017ML, MCP:QFN28-ML_6X6MM
- removed IC2: TPS70933DBV, tps709xx_10:SOT23-5
- removed IC3: LM2596S, national-semiconductor:TO263-5
- removed IC4: ACS758ECB-200B-PFF-T, allegro-2:CB-PFF
- removed J1, J3: (no value), SparkFun-Connectors:1X04
- removed J4: (no value), SparkFun-Connectors:1X05
- removed L2: CDRH127/LD, inductor-sumida:CDRH127/LD
- removed L4: 100, SparkFun-Coils:SRN6045
- removed LED1, LED2, LED3: Red, led:SML0603
- removed ON: Button, SparkFun-Switches:TACTILE_SWITCH_SMD_RIGHT_ANGLE
- removed PAD1, PAD10, PAD11, PAD12, PAD2, PAD3, PAD4, PAD5, PAD6, PAD7, PAD8, PAD9: (no value), wirepad:SMD2,54-5,08
- removed SW: (no value), SparkFun-Switches:SWITCH_SPST_SMD_A
- removed T1, T2: (no value), transistor:SOT23-BEC
- removed U$16, U$18: TOF+SHARP, TOF+SHARP:TOF+SHARP_V1
- removed U$17, U$36, U$37, U$38: XT60, XT60:XT60
- removed U$19, U$20, U$27, U$29: TOF-SHARP, TOF+SHARP:TOF+SHARP_V2
- removed U$30: SUPER_DUPER_GUZICZEK, SuperDuperGuziczek:SUPER_DUPER_GUZICZEK
- removed U$32: IR_SW, IR_SW:IR_SW
- removed U$33: TLA2024, TLA2024:X2QFN
- removed U$34: HM-11, hm-11:HM-11
- removed U$35: MP2307, MP2307:SOIC8N
- removed U$39: STM32F030F4, STM32L0:TSSOP20
- removed U1: VL53L0X, microbuilder:LGA12_ST
- removed U3: STM32F10XRXT6, stm32:TQFP64
- added R3: 100R, resistor:R0603
- C10: value 10uF -> 1uF; device rcl:153CLV-0605 -> rcl:C0603
- C11, C8, C9: value (none) -> 1uF; device rcl:153CLV-0810 -> rcl:C0603
- C12, C15: value (none) -> 1000pF; device rcl:153CLV-0810 -> rcl:C0603
- C16, C17: value (none) -> 4.7uF; device rcl:153CLV-0810 -> rcl:C0805
- C4, C7: value (none) -> 0.047uF; device rcl:153CLV-0810 -> rcl:C0603
- R2: value 100k -> 10k
- U$12: value CSD17573Q5B -> STM32G473CC; device CSD_Mosfet:Q5B -> STM32G473CC:VFQFPN36
- U$13: value CSD17573Q5B -> DRV8305; device CSD_Mosfet:Q5B -> drv8305lbr:S-PQFP-G48
- U$14, U$15: value TOF+SHARP -> MOLEG_REC_8X0.4MM; device TOF+SHARP:TOF+SHARP_V1 -> MOLEX:REC
- moved R2 134.1 mm to (33.1, 22.7), flipped to the top, turned to 180 degrees
- moved C10 132.0 mm to (48.0, 8.90), flipped to the top, turned to 270 degrees
- moved U$13 126.9 mm to (40.1, 16.4), flipped to the top
- moved U$14 123.4 mm to (34.3, 6.18), flipped to the top, turned to 0 degrees
- moved U$15 113.9 mm to (40.4, 3.94), flipped to the top
- moved U$12 110.1 mm to (54.3, 24.1), flipped to the top, turned to 0 degrees
- moved C8 78.1 mm to (31.4, 15.2), turned to 90 degrees
- moved C9 71.4 mm to (42.0, 21.8), turned to 0 degrees
- moved C7 70.6 mm to (42.9, 12.3), turned to 90 degrees
- moved C4 65.0 mm to (42.9, 15.2), turned to 270 degrees
- moved C17 56.2 mm to (44.3, 12.5), turned to 270 degrees
- moved C11 55.4 mm to (31.7, 20.3), turned to 180 degrees
- moved C12 53.9 mm to (31.4, 12.3), turned to 270 degrees
- moved C15 49.1 mm to (30.3, 12.3), turned to 270 degrees
- moved C16 34.7 mm to (44.3, 15.7), turned to 90 degrees
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Connections:
- removed net 11.1V: 0026.2, PAD1.1, PAD5.1
- removed net 14.8V: 0029.2, PAD2.1, PAD4.1
- removed net 3.7V: 0023.2, PAD12.1, PAD9.1
- removed net 3V3: 0004.1, C22.2, C25.1, C26.+, J1.3, L4.2, U$32.VCC, U$34.VCC
- removed net 3V3_L0: 0012.1, C33.+, IC2.5, J4.1, R2.1, U$39.16, U$39.5
- removed net 5V: 0032.1, C20.+, C29.1, C35.2, IC4.1, J1.4, L2.2, U$14.5V, U$15.5V, U$16.5V, U$18.5V, U$19.5V, U$20.5V, U$27.5V, U$29.5V
- removed net 7.4V: 0024.2, C30.+, IC2.1, PAD11.1, PAD3.1, PAD6.1, PAD7.1
- removed net A11.1: 0026.1, 0027.2, U$39.8
- removed net A14.8: 0028.2, 0029.1, U$39.9
- removed net A3.7: 0007.2, 0023.1, U$39.6
- removed net A7.4: 0024.1, 0025.2, U$39.7
- removed net ACURR: 0030.1, 0031.1, U$39.10
- removed net AVDD: U1.11
- removed net AVDDVCSEL: U1.1
- removed net AVSSVCSEL: U1.2
- removed net BAT-: 0007.1, 0008.1, 0010.1, 0011.2, 0025.1, 0027.1, 0028.1, 0030.2, C21.1, C30.-, C33.-, IC2.2, J4.3, LED3.C, PAD10.1, PAD8.1, T1.E, U$12.S1, U$12.S2, U$12.S3, U$13.S1, U$13.S2, U$13.S3, U$30.T1, U$30.T2, U$39.1, U$39.15
- removed net BS: C18.1, U$35.1
- removed net BUTTON_L0: LED3.A, ON.1, U$39.13
- removed net COMP: C24.1, U$35.6
- removed net CURR: 0031.2, IC4.3
- removed net EN: 0006.1, U$35.7
- removed net FB: 0003.2, 0004.2, U$35.5
- removed net GATE: U$13.G
- removed net GPIO_1: U$14.GPIO
- removed net GPIO_2: U$15.GPIO
- removed net GPIO_3: U$16.GPIO
- removed net GPIO_4: U$18.GPIO
- removed net GPIO_5: U$19.GPIO
- removed net GPIO_6: U$20.GPIO
- removed net GPIO_7: U$27.GPIO
- removed net GPIO_8: U$29.GPIO
- removed net KILL: IC1.22, U$32.KILL
- removed net LED_L0: LED2.A, U$39.12
- removed net MOSFET: 0009.2, U$39.14
- removed net N$1: 0032.2, 0033.1, C35.1, IC3.4
- removed net N$29: 0022.1, T1.C, T2.B
- removed net N$41: IC1.3
- removed net N$42: IC1.4
- removed net N$44: IC1.23
- removed net N$46: IC1.24
- removed net N$52: 0010.2, LED2.C
- removed net N$54: 0012.2, ON.2
- removed net N$58: U$39.11
- removed net N$6: 0008.2, 0009.1, T1.B
- removed net N$87: 0013.1, LED1.A
- removed net N$89: 0011.1, T2.C, U$12.G
- removed net NRST_L0: C21.2, J4.5, R2.2, U$30.T3, U$30.T4, U$39.4
- removed net OUT: D1.C, IC3.2, L2.1
- removed net RX: U$34.UART_RX
- removed net SAFE_SW: SW.1, T2.E
- removed net SCL_L: U$14.SCL, U$15.SCL, U$16.SCL, U$18.SCL, U3.58
- removed net SCL_L0: J1.1, U$39.17
- removed net SCL_R: U$19.SCL, U$20.SCL, U$27.SCL, U$29.SCL, U3.29
- removed net SDA_L: U$14.SDA, U$15.SDA, U$16.SDA, U$18.SDA, U3.59
- removed net SDA_L0: J1.2, U$39.18
- removed net SDA_R: U$19.SDA, U$20.SDA, U$27.SDA, U$29.SDA, U3.30
- removed net SHARP_1: IC1.17, U$14.SHARP
- removed net SHARP_2: IC1.18, U$15.SHARP
- removed net SHARP_3: IC1.19, U$16.SHARP
- removed net SHARP_4: IC1.20, U$18.SHARP
- removed net SHARP_5: U$19.SHARP
- removed net SHARP_6: U$20.SHARP
- removed net SHARP_7: U$27.SHARP
- removed net SHARP_8: U$29.SHARP
- removed net SS: C27.1, U$35.8
- removed net START: IC1.21, U$32.START
- removed net SW: C18.2, L4.1, U$35.3
- removed net SWCLK_L0: J4.2, U$39.20
- removed net SWDIO_L0: J4.4, U$39.19
- removed net TX: U$34.UART_TX
- removed net VBAT: U3.1
- removed net VDD: IC1.5
- removed net VDDA: U3.13
- removed net VDD_1: U3.32
- removed net VDD_2: U3.48
- removed net VDD_3: U3.64
- removed net VDD_4: U3.19
- removed net VIN: 0006.2, 0013.2, 0022.2, C10.+, C11.+, C12.+, C15.+, C16.+, C17.+, C23.+, C28.1, C4.+, C7.+, C8.+, C9.+, SW.2, U$17.+, U$35.2, U$36.+, U$37.+, U$38.+
- removed net VIN1: C19.+, IC3.1
- removed net VSS: IC1.6
- removed net VSSA: U3.12
- removed net VSS_1: U3.31
- removed net VSS_2: U3.47
- removed net VSS_3: U3.63
- removed net VSS_4: U3.18
- removed net XSHUT_1: IC1.25, U$14.XSHUT
- removed net XSHUT_2: IC1.26, U$15.XSHUT
- removed net XSHUT_3: IC1.27, U$16.XSHUT
- removed net XSHUT_4: IC1.28, U$18.XSHUT
- removed net XSHUT_5: U$19.XSHUT
- removed net XSHUT_6: U$20.XSHUT
- removed net XSHUT_7: U$27.XSHUT
- removed net XSHUT_8: U$29.XSHUT
- removed net XXX: IC1.1
- new net +3V3_: C11.1, R2.2
- new net ENGATE_: U$13.1-EN_GATE
- new net GH_A_: U$13.36-GH_A, U$15.POWER_2
- new net GH_B_: U$13.29-GH_B, U$14.POWER_4
- new net GH_C_: U$13.28_GH_C, U$14.POWER_3
- new net GL_A_: U$13.33-GL_A, U$15.POWER_3
- new net GL_B_: U$13.32-GL_B, U$14.POWER_2
- new net GL_C_: U$13.25-GL_C, U$14.POWER_1
- new net GND_: C10.2, C11.2, C16.2, C8.2, C9.2, U$13.14-GND1, U$13.21-SN2, U$13.22-SP2, U$13.45-GND2, U$13.9-NSCS, U$13.POWERPAD, U$14.PAD_1, U$14.PAD_2, U$14.PAD_3, U$14.PAD_4, U$15.PAD_1, U$15.PAD_2, U$15.PAD_3, U$15.PAD_4, U$15.POWER_4
- new net INH_A_: U$13.2-INHA
- new net INH_B_: U$13.4-INHB
- new net INH_C_: U$13.6-INHC
- new net INL_A_: U$13.3-INLA
- new net INL_B_: U$13.5-INLB
- new net INL_C_: U$13.7-INLC
- new net N$30: C9.1, U$13.46-DVDD
- new net N$31: C8.1, U$13.15-AVDD
- new net N$32: C10.1, U$13.37-VCP_LSD
- new net N$33: C4.2, U$13.42-CP1L
- new net N$35: C7.2, U$13.40-CP2L
- new net N$36: C7.1, U$13.39-CP2H
- new net N$38: R3.1, U$13.44-VDRAIN
- new net N$39: C17.2, U$13.38-VCPH
- new net NFAULT_: R2.1, U$13.8-NFAULT
- new net PWRGD_: U$13.13-PWRGD
- new net SCLK_: U$13.12-SCLK
- new net SDI_: U$13.10-SDI
- new net SDO_: U$13.11-SDO
- new net SH_A_: U$13.35-SH_A, U$15.SIGNAL_1
- new net SH_B_: U$13.30-SH_B, U$15.SIGNAL_2
- new net SH_C_: U$13.27-SH_C, U$14.SIGNAL_4
- new net SL_A_: C12.1, U$13.23-SN1, U$13.34-SL_A, U$15.SIGNAL_3
- new net SL_B_: U$13.31-SL_B, U$15.SIGNAL_4
- new net SL_C_: C15.1, U$13.19-SN3, U$13.26-SL_C, U$14.SIGNAL_1
- new net SO1_: U$13.16-SO1
- new net SO3_: U$13.18-SO3
- new net SP_A_: C12.2, U$13.24-SP1, U$14.SIGNAL_2
- new net SP_C_: C15.2, U$13.20-SP3, U$14.SIGNAL_3
- new net VMOTOR_: C16.1, C17.1, R3.2, U$13.41-PVDD, U$15.POWER_1
- new net WAKE_: U$13.47-WAKE
- net GND: no longer 0003.1, 0005.1, 0033.2, C10.-, C11.-, C12.-, C15.-, C16.-, C17.-, C19.-, C20.-, C22.1, C23.-, C25.2, C26.-, C27.2, C28.2, C29.2, C4.-, C7.-, C8.-, C9.-, D1.A, IC3.3, IC4.2, LED1.C, U$12.D1, U$12.D2, U$12.D3, U$12.D4, U$12.D5, U$13.D1, U$13.D2, U$13.D3, U$13.D4, U$13.D5, U$14.GND\, U$15.GND\, U$16.GND\, U$17.-, U$18.GND\, U$19.GND\, U$20.GND\, U$27.GND\, U$29.GND\, U$32.GND, U$34.GND, U$35.4, U$35.PAD, U$36.-, U$37.-, U$38.-, U1.12, U1.3, U1.4, U1.6
- net N$34: now also C4.1, U$13.43-CP1H; no longer 0005.2, C24.2
- net N$40: now also U$13.48-VREG; no longer IC1.2
Routing:
- net VMOTOR_TOP: track 14.4 -> 12.8 mm
Other:
- board size 271.8 x 122.6 mm -> 26.6 x 48.3 mm
- board text removed: "0V"
- board text removed: "3.7V"
- board text removed: "7.4V"
- board text removed: "I2C isolator :D"
- board text removed: "bez wycinanek"
- board text removed: "dioda na czujniku do skarpa"
- board text removed: "moze ten kondensatorek dla ldo sie zmiesci XDD"
- board text removed: "rezystorki do masy na szumy dla sharpow"
- board text removed: "tedy polaczenia beda"
- board text removed: "wazna zmiana tu ->"
