File: 1.UberDirver v3 STM32F103/Schemat/Schematic.brd (EAGLE design)
At the start: 59 x 42.1 mm, 86 parts, among them U2 STM32F10XTXU6HS

Commit message: Inzynier zrobiony
dodano wersje 3
Parts:
- removed 0001: 34.8kR, rcl:R0402
- removed 0015: 5mohm, resistor:R2512
- removed C49: 100nF, rcl:R0402
- removed C67, C68, C69: 220uf, rcl:150CLZ-0810
- added C24\, C25, C26, C27: 22uF, rcl:C1206
- added C28: 220uf, rcl:150CLZ-0810
- added C48: (no value), rcl:C025-040X050
- added D2, D3, D4, D5: (no value), adafruit:SOD-123FL
- added L1: 1mH, resistor:R0603
- added L2, L3, L4, R21, R22, R23: (no value), rcl:0204/5
- added PAD_A1, PAD_A2: (no value), wirepad:SMD2,54-5,08
- added Q10, Q11, Q12, Q13, Q14, Q7, Q8, Q9: CSD17573Q5B, CSD_Mosfet:Q5B
- added R10: 10k, rcl:R0402
- added R11: 100R, resistor:R0603
- C1, C2, C3: value 100nF -> 1nF
- C10, C11: value 220uf -> 0.047uF; device rcl:150CLZ-0810 -> rcl:R0402
- C12: value 220uf -> 4.7uF; device rcl:150CLZ-0810 -> rcl:C0805
- C14: value 4.7uF -> 1nF; device rcl:C0805 -> rcl:R0402
- C15, C4: value 220uf -> 1nF; device rcl:150CLZ-0810 -> rcl:R0402
- C16, C18, C20, C22: value 220uf -> 100nF; device rcl:150CLZ-0810 -> rcl:R0402
- C17, C19, C21, C23: value 220uf -> 4.7uF; device rcl:150CLZ-0810 -> rcl:R0402
- C24: value 220uf -> (none); device rcl:150CLZ-0810 -> rcl:C025-040X050
- C29, C35, C37, C40: value 4.7uF -> 220uf; device rcl:R0402 -> rcl:150CLZ-0810
- C30, C33, C41, C43: value 22uF -> 220uf; device rcl:C1206 -> rcl:150CLZ-0810
- C31, C32: value 0.047uF -> 220uf; device rcl:R0402 -> rcl:150CLZ-0810
- C34, C36, C38, C39: value 1uF -> 220uf; device rcl:R0402 -> rcl:150CLZ-0810
- C42, C44: value 1nF -> 220uf; device rcl:R0402 -> rcl:150CLZ-0810
- C45, C46, C47: value 100nF -> 220uf; device rcl:R0402 -> rcl:150CLZ-0810
- C6: value 100nF -> 1uF
- C7, C8, C9: value 220uf -> 1uF; device rcl:150CLZ-0810 -> rcl:R0402
- R1: value 180nH -> 100k; device resistor:R0603 -> rcl:R0402
- R13: value 100R -> 5mohm; device resistor:R0603 -> resistor:R2512
- R24: value 10k -> (none); device rcl:R0402 -> rcl:0204/5
- R3, R5, R7: value 34.8kR -> 100k
- moved R24 80.2 mm to (-20.4, -57.1), turned to 90 degrees
- moved C24 76.9 mm to (-15.3, -57.4), flipped to the top, turned to 270 degrees
- moved C36 33.8 mm to (9.11, 32.1), flipped to the top
- moved C9 33.8 mm to (35.6, 11.2), flipped to the bottom
- moved C44 30.3 mm to (52.0, 32.1), turned to 90 degrees
- moved C47 28.7 mm to (52.0, 22.1), flipped to the bottom, turned to 270 degrees
- moved C22 28.7 mm to (26.6, 8.78), flipped to the top, turned to 90 degrees
- moved C39 28.2 mm to (9.10, 22.0), turned to 270 degrees
- moved C10 27.6 mm to (35.5, 14.1), flipped to the bottom, turned to 0 degrees
- moved C45 26.6 mm to (9.11, 32.1), flipped to the bottom
- moved C16 26.6 mm to (31.3, 15.4), flipped to the top, turned to 0 degrees
- moved C11 25.2 mm to (35.5, 13.0), flipped to the bottom, turned to 0 degrees
- moved C29 24.5 mm to (52.0, 32.1), turned to 90 degrees
- moved C34 24.2 mm to (17.7, 32.1), flipped to the top, turned to 90 degrees
- moved C35 24.1 mm to (43.4, 32.1), turned to 90 degrees
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- renumbered 0002 to R2, 0014 to R12, 0016 to R3, 0017 to R4, 0018 to R7, 0019 to R8, 0020 to R5, 0021 to R6, LED9 to D1, MOTOR_PAD_C to PAD_C, M_A to PAD_A, M_B to PAD_B, R16 to R9, U$22 to Q3, U$23 to Q4, U$24 to Q1, U$25 to Q2, U$26 to Q5, U$28 to Q6
Connections:
- new net +VCC: Q10.D, Q11.D, Q9.D
- new net N$15: PAD_A1.1, R21.2
- new net N$17: C48.1, D2.A, D3.C, R21.1, R22.2
- new net N$18: C48.2, D3.A, R22.1
- new net N$19: PAD_A2.1, R23.2
- new net N$24: D2.C
- new net N$25: C24.1, D4.A, D5.C, R23.1, R24.2
- new net N$26: C24.2, D5.A, R24.1
- new net N$27: D4.C
- new net N$29: Q7.S, Q8.D
- new net N$31: Q8.G
- new net N$32: Q7.G
- new net N$41: L2.1, Q12.D, Q9.S
- new net N$42: L4.1, Q10.S, Q13.D
- new net N$43: L3.1, Q11.S, Q14.D
- new net N$45: L2.2, L3.2, L4.2
- new net VCC: Q7.D
- net +3V3: now also C18.1, C19.1, C20.1, C21.1, C22.1, C23.1, C6.1, L1.2; no longer C1.1, C2.1, C29.1, C35.1, C37.1, C39.1, C49.1, R1.2
- net ADC_VA: now also C4.1; no longer C45.1
- net ADC_VB: now also C3.1; no longer C46.1
- net ADC_VC: now also C2.1; no longer C47.1
- net ADC_VMOT: now also C1.1, R1.1; no longer 0001.1, C6.1
- net GND: now also C16.2, C17.2, C18.2, C19.2, C20.2, C21.2, C22.2, C23.2, C24\.2, C25.2, C26.2, C27.2, C28.-, C29.-, C30.-, C31.-, C32.-, C33.-, C34.-, C35.-, C36.-, C37.-, C38.-, C39.-, C4.2, C40.-, C41.-, C42.-, C43.-, C44.-, C45.-, C46.-, C47.-, C7.2, C8.2, C9.2, Q12.S, Q13.S, Q14.S, Q8.S, R10.1, R13.1; no longer 0015.1, C10.-, C11.-, C12.-, C15.-, C16.-, C17.-, C18.-, C19.-, C20.-, C21.-, C22.-, C23.-, C24.-, C29.2, C30.2, C33.2, C34.2, C35.2, C36.2, C37.2, C38.2, C39.2, C4.-, C40.2, C41.2, C43.2, C45.2, C46.2, C47.2, C49.2, C67.-, C68.-, C69.-, C7.-, C8.-, C9.-, R24.1
- net GND_A: now also C14.2; no longer C42.2
- net GND_C: now also C15.2; no longer C44.2
- net N$10: now also C9.1; no longer C36.1
- net N$12: now also C8.1; no longer C34.1
- net N$13: now also C7.1; no longer C38.1
- net N$14: now also C11.2; no longer C31.2
- net N$16: now also C11.1; no longer C31.1
- net N$2: now also C16.1, C17.1, L1.1; no longer C3.1, C40.1, R1.1
- net N$20: now also C10.2; no longer C32.2
- net N$21: now also C10.1; no longer C32.1
- net N$22: now also R11.1; no longer R13.1
- net N$23: now also C12.2; no longer C14.2
- net N$81: now also R10.2; no longer R24.2
- net SL_A: now also C14.1; no longer C42.1
- net SL_C: now also C15.1, R13.2; no longer 0015.2, C44.1
- net VMOTOR: now also C12.1, C24\.1, C25.1, C26.1, C27.1, C28.+, C29.+, C30.+, C31.+, C32.+, C33.+, C34.+, C35.+, C36.+, C37.+, C38.+, C39.+, C40.+, C41.+, C42.+, C43.+, C44.+, C45.+, C46.+, C47.+, R1.2, R11.2; no longer 0001.2, C10.+, C11.+, C12.+, C14.1, C15.+, C16.+, C17.+, C18.+, C19.+, C20.+, C21.+, C22.+, C23.+, C24.+, C30.1, C33.1, C4.+, C41.1, C43.1, C67.+, C68.+, C69.+, C7.+, C8.+, C9.+, R13.2
Routing:
- net N$28: track 0.00 -> 73.2 mm
- net N$25: track 0.00 -> 61.1 mm
- net N$17: track 0.00 -> 41.9 mm
- net N$18: track 0.00 -> 40.3 mm
- net N$26: track 0.00 -> 19.7 mm, vias 0 -> 2
- net N$19: track 0.00 -> 5.94 mm
- net N$15: track 0.00 -> 5.45 mm
- net N$27: track 0.00 -> 4.23 mm
- net N$24: track 0.00 -> 3.08 mm
Other:
- board size 59 x 42.1 mm -> 89.6 x 77.9 mm
- board text added: "3.3V"
- board text added: "A"
- board text added: "B"
- board text added: "DOBRZE"
- board text added: "Mikrokontroler"
- board text added: "ŹLE"
